File: schematic/sensorboard.brd (EAGLE design)
At the start: 34.5 x 57 mm, 49 parts, among them J1 UART Connection, J2 455-1750-1-ND, Q1 MMSS8050-L-TP, Q2 MMSS8050-L-TP, Q3 MMSS8050-L-TP, U1 ATMEGA328P_TQFP, U2 XC6206P302, U4 S16-L221D, Y1 8MHz

Commit message: added more debug options
Parts:
- moved R20 51.1 mm to (1.02, 48.0), flipped to the bottom, turned to 270 degrees
- moved C1 0.51 mm to (2.18, 49.3)
Routing:
- net VCC: track 146.4 -> 147.6 mm
- net N$10: track 29.0 -> 30.0 mm
- net DTR: track 18.4 -> 17.9 mm
Changed lines of the file:
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@@
 <?xml version="1.0" encoding="utf-8"?>
 <!DOCTYPE eagle SYSTEM "eagle.dtd">
-<eagle version="9.6.1">
+<eagle version="9.6.2">
 <drawing>
 <settings>
@@
 <layer number="25" name="tNames" color="7" fill="1" visible="yes" active="yes"/>
 <layer number="26" name="bNames" color="7" fill="1" visible="yes" active="yes"/>
-<layer number="27" name="tValues" color="7" fill="1" visible="no" active="yes"/>
+<layer number="27" name="tValues" color="7" fill="1" visible="yes" active="yes"/>
 <layer number="28" name="bValues" color="7" fill="1" visible="no" active="yes"/>
 <layer number="29" name="tStop" color="7" fill="3" visible="no" active="yes"/>
@@
 </layers>
 <board>
-<fusionsync huburn="a.YnVzaW5lc3M6bXlnbXgyMzIxMw" projecturn="a.YnVzaW5lc3M6bXlnbXgyMzIxMyNEMjAyMDA1MjAzMDAxMDA1NTY" f3durn="urn:adsk.wipprod:dm.lineage:RlprBCnbRoK6DUTxJZNohQ" pcbguid="a0c7e5cc-de5c-430a-88de-9707ba0d7ca6" lastpulledtime="" lastsyncedchangeguid="2950f385-ff89-3442-d435-59eeb59bf3b9" latestrevisionid="e00f23df-46e1-439b-82a3-be38e5a88ebf" lastsyncedrevisionid="e00f23df-46e1-439b-82a3-be38e5a88ebf" lastboardhashguid="2950f385-ff89-3442-d435-59eeb59bf3b9" lastpushedtime="2021-04-07T09:00:36Z" linktopcb3d="%12"/>
+<fusionsync huburn="a.YnVzaW5lc3M6bXlnbXgyMzIxMw" projecturn="a.YnVzaW5lc3M6bXlnbXgyMzIxMyNEMjAyMDA1MjAzMDAxMDA1NTY" f3durn="urn:adsk.wipprod:dm.lineage:RlprBCnbRoK6DUTxJZNohQ" pcbguid="a0c7e5cc-de5c-430a-88de-9707ba0d7ca6" lastpulledtime="" lastsyncedchangeguid="2950f385-ff89-3442-d435-59eeb59bf3b9" latestrevisionid="e00f23df-46e1-439b-82a3-be38e5a88ebf" lastsyncedrevisionid="e00f23df-46e1-439b-82a3-be38e5a88ebf" lastboardhashguid="2950f385-ff89-3442-d435-59eeb59bf3b9" lastpushedtime="2021-04-07T09:00:36Z" linktopcb3d="false"/>
 <plain>
 <circle x="17.018" y="40.386" radius="5.1" width="0.254" layer="21"/>
@@
 </autorouter>
 <elements>
-<element name="C1" library="rcl" library_urn="urn:adsk.eagle:library:334" package="C0402" package3d_urn="urn:adsk.eagle:package:23626/2" value="100n" x="1.676" y="49.251" smashed="yes" rot="MR270">
-<attribute name="NAME" x="1.041" y="49.886" size="1.016" layer="26" rot="MR270"/>
-<attribute name="POPULARITY" value="18" x="44.856" y="13.691" size="1.778" layer="28" rot="MR270" display="off"/>
-<attribute name="SPICEPREFIX" value="C" x="44.856" y="13.691" size="1.778" layer="28" rot="MR270" display="off"/>
+<element name="C1" library="rcl" library_urn="urn:adsk.eagle:library:334" package="C0402" package3d_urn="urn:adsk.eagle:package:23626/2" value="100n" x="2.184" y="49.251" smashed="yes" rot="MR270">
+<attribute name="NAME" x="2.007" y="50.952" size="0.6096" layer="26" rot="MR90"/>
+<attribute name="POPULARITY" value="18" x="45.364" y="13.691" size="1.778" layer="28" rot="MR270" display="off"/>
+<attribute name="SPICEPREFIX" value="C" x="45.364" y="13.691" size="1.778" layer="28" rot="MR270" display="off"/>
 </element>
 <element name="C2" library="rcl" library_urn="urn:adsk.eagle:library:334" package="C0402" package3d_urn="urn:adsk.eagle:package:23626/2" value="10u" x="7.874" y="49.022" smashed="yes" rot="MR90">
@@
 <attribute name="SPICEPREFIX" value="C" x="5.842" y="34.798" size="1.016" layer="28" rot="MR270" display="off"/>
 </element>
-<element name="R20" library="rcl" library_urn="urn:adsk.eagle:library:334" package="R0402" package3d_urn="urn:adsk.eagle:package:23547/3" value="10k" x="-4.318" y="-2.794" smashed="yes">
-<attribute name="NAME" x="-4.953" y="-2.159" size="1.27" layer="25"/>
-<attribute name="POPULARITY" value="0" x="-4.318" y="-2.794" size="1.778" layer="27" display="off"/>
-<attribute name="SPICEPREFIX" value="R" x="-4.318" y="-2.794" size="1.778" layer="27" display="off"/>
-<attribute name="VALUE" x="-4.953" y="-4.699" size="1.27" layer="27"/>
+<element name="R20" library="rcl" library_urn="urn:adsk.eagle:library:334" package="R0402" package3d_urn="urn:adsk.eagle:package:23547/3" value="10k" x="1.016" y="48.006" smashed="yes" rot="MR270">
+<attribute name="NAME" x="0.889" y="49.149" size="0.6096" layer="26" rot="MR90"/>
+<attribute name="POPULARITY" value="0" x="1.016" y="48.006" size="1.778" layer="28" rot="MR270" display="off"/>
+<attribute name="SPICEPREFIX" value="R" x="1.016" y="48.006" size="1.778" layer="28" rot="MR270" display="off"/>
+<attribute name="VALUE" x="2.921" y="48.641" size="1.27" layer="28" rot="MR270"/>
 </element>
 </elements>
@@
 <wire x1="9.074" y1="26.092" x2="9.074" y2="27.1526" width="0.4064" layer="16"/>
 <contactref element="R20" pad="2"/>
-<wire x1="-3.818" y1="-2.794" x2="9.06000625" y2="15.91800625" width="0" layer="19" extent="1-1"/>
+<wire x1="1.016" y1="47.506" x2="1.0414" y2="47.4806" width="0.254" layer="16"/>
+<wire x1="1.0414" y1="47.4806" x2="1.0414" y2="46.355" width="0.254" layer="16"/>
 </signal>
 <signal name="DTR">
@@
 <wire x1="14.732" y1="50.038" x2="14.986" y2="50.292" width="0.254" layer="16"/>
 <wire x1="14.986" y1="50.292" x2="14.986" y2="54.356" width="0.254" layer="16"/>
-<wire x1="1.676" y1="49.901" x2="2.4026" y2="49.9006" width="0.254" layer="16"/>
-<wire x1="3.302" y1="50.8" x2="2.4026" y2="49.9006" width="0.254" layer="16"/>
+<wire x1="2.184" y1="49.901" x2="2.402878125" y2="49.900878125" width="0.254" layer="16"/>
+<wire x1="3.302" y1="50.8" x2="2.402878125" y2="49.900878125" width="0.254" layer="16"/>
 </signal>
 <signal name="TX">
@@
 <contactref element="U1" pad="29"/>
 <contactref element="C1" pad="2"/>
-<wire x1="1.676" y1="48.601" x2="1.6764" y2="47.8536" width="0.254" layer="16"/>
-<wire x1="1.6764" y1="47.8536" x2="4.064" y2="45.466" width="0.254" layer="16"/>
+<wire x1="2.184" y1="48.601" x2="2.184671875" y2="47.345328125" width="0.254" layer="16"/>
+<wire x1="2.184671875" y1="47.345328125" x2="4.064" y2="45.466" width="0.254" layer="16"/>
 <wire x1="4.064" y1="40.386" x2="1.5748" y2="37.8968" width="0.254" layer="16"/>
 <wire x1="2.14" y1="23.26" x2="3.5814" y2="23.26" width="0.254" layer="16"/>
@@
 <wire x1="1.5748" y1="23.8252" x2="2.14" y2="23.26" width="0.254" layer="16"/>
 <contactref element="R20" pad="1"/>
-<wire x1="-4.818" y1="-2.794" x2="3.5814" y2="23.26" width="0" layer="19" extent="1-16"/>
+<wire x1="1.016" y1="48.506" x2="1.111" y2="48.601" width="0.254" layer="16"/>
+<wire x1="1.111" y1="48.601" x2="2.184" y2="48.601" width="0.254" layer="16"/>
 </signal>
 <signal name="MOSI">
